File: FireFly/FireFly.brd (EAGLE design)
At the start: 20.3 x 44.1 mm, 13 parts

Commit message: update
Routing:
- net N$9: track 10.2 -> 11.6 mm
- net N$15: track 30.0 -> 29.3 mm
- net N$10: track 31.5 -> 30.8 mm
- net N$13: track 29.6 -> 30.4 mm
- net N$6: vias 6 -> 4
Changed lines of the file:
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@@
 <?xml version="1.0" encoding="utf-8"?>
 <!DOCTYPE eagle SYSTEM "eagle.dtd">
-<eagle version="9.5.2">
+<eagle version="9.6.2">
 <drawing>
 <settings>
@@
 <via x="20.32" y="31.75" extent="1-16" drill="0.35"/>
 <wire x1="20.32" y1="31.75" x2="21.59" y2="33.02" width="0.6096" layer="1"/>
-<wire x1="19.05" y1="25.4" x2="19.05" y2="30.48" width="0.6096" layer="16"/>
-<wire x1="19.05" y1="30.48" x2="20.32" y2="31.75" width="0.6096" layer="16"/>
+<wire x1="19.05" y1="25.4" x2="19.05" y2="27.94" width="0.6096" layer="16"/>
+<wire x1="20.32" y1="29.21" x2="19.05" y2="27.94" width="0.6096" layer="16"/>
+<wire x1="20.32" y1="29.21" x2="20.32" y2="31.75" width="0.6096" layer="16"/>
 <wire x1="25.4" y1="31.75" x2="20.32" y2="31.75" width="0.6096" layer="16"/>
 <wire x1="10.16" y1="36.83" x2="15.24" y2="36.83" width="0.6096" layer="16"/>
@@
 <vertex x="26.67" y="43.18"/>
 </polygon>
-<via x="15.24" y="30.48" extent="1-16" drill="0.35"/>
-<via x="13.97" y="8.89" extent="1-16" drill="0.35"/>
-<via x="11.43" y="2.54" extent="1-16" drill="0.35"/>
+<via x="13.97" y="10.16" extent="1-16" drill="0.35"/>
 <via x="24.13" y="2.54" extent="1-16" drill="0.35"/>
 <via x="15.24" y="19.05" extent="1-16" drill="0.35"/>
@@
 <contactref element="RELAY" pad="3"/>
 <contactref element="JP7" pad="13"/>
-<wire x1="25.4" y1="8.89" x2="22.86" y2="8.89" width="0.508" layer="1"/>
-<wire x1="22.86" y1="8.89" x2="21.59" y2="7.62" width="0.508" layer="1"/>
-<wire x1="21.59" y1="7.62" x2="17.78" y2="7.62" width="0.508" layer="1"/>
+<wire x1="25.4" y1="8.89" x2="24.13" y2="7.62" width="0.508" layer="1"/>
+<wire x1="24.13" y1="7.62" x2="17.78" y2="7.62" width="0.508" layer="1"/>
 <wire x1="17.78" y1="7.62" x2="16.51" y2="8.89" width="0.508" layer="1"/>
 <wire x1="16.51" y1="8.89" x2="16.51" y2="10.16" width="0.508" layer="1"/>
@@
 <contactref element="JP7" pad="11"/>
 <via x="17.78" y="30.48" extent="1-16" drill="0.35"/>
-<wire x1="13.97" y1="33.02" x2="16.51" y2="33.02" width="0.508" layer="1"/>
-<wire x1="16.51" y1="33.02" x2="17.78" y2="31.75" width="0.508" layer="1"/>
-<wire x1="17.78" y1="31.75" x2="17.78" y2="30.48" width="0.508" layer="1"/>
+<wire x1="13.97" y1="33.02" x2="15.24" y2="33.02" width="0.508" layer="1"/>
+<wire x1="15.24" y1="33.02" x2="17.78" y2="30.48" width="0.508" layer="1"/>
 <via x="17.78" y="12.7" extent="1-16" drill="0.35"/>
 <wire x1="17.78" y1="30.48" x2="17.78" y2="12.7" width="0.508" layer="16"/>
@@
 <wire x1="17.272" y1="13.462" x2="15.24" y2="11.43" width="0.2032" layer="1"/>
 <wire x1="15.24" y1="11.43" x2="15.24" y2="3.81" width="0.2032" layer="1"/>
-<wire x1="15.24" y1="3.81" x2="16.51" y2="2.54" width="0.2032" layer="1"/>
 <wire x1="16.51" y1="2.54" x2="17.03" y2="2.54" width="0.2032" layer="1"/>
 <wire x1="20.828" y1="13.462" x2="17.272" y2="13.462" width="0.2032" layer="1"/>
 <wire x1="22.34" y1="13.45" x2="25.4" y2="16.51" width="0.2032" layer="1"/>
+<wire x1="15.24" y1="3.81" x2="16.51" y2="2.54" width="0.2032" layer="1"/>
 </signal>
 <signal name="N$12">
@@
 <contactref element="MSG" pad="A"/>
 <contactref element="JP7" pad="8"/>
-<wire x1="25.4" y1="21.59" x2="23.2156" y2="19.4056" width="0.2032" layer="1"/>
-<wire x1="23.2156" y1="19.4056" x2="23.2156" y2="18.9027" width="0.2032" layer="1"/>
+<wire x1="25.4" y1="21.59" x2="24.13" y2="21.59" width="0.2032" layer="1"/>
+<wire x1="24.13" y1="21.59" x2="23.2156" y2="20.6756" width="0.2032" layer="1"/>
+<wire x1="23.2156" y1="20.6756" x2="23.2156" y2="18.9027" width="0.2032" layer="1"/>
 <wire x1="15.61593125" y1="17.78" x2="15.24" y2="17.78" width="0.2032" layer="1"/>
 <wire x1="16.24813125" y1="17.1478" x2="15.61593125" y2="17.78" width="0.2032" layer="1"/>
@@
 <wire x1="21.59" y1="20.32" x2="21.59" y2="15.24" width="0.6096" layer="16"/>
 <wire x1="21.59" y1="25.4" x2="21.59" y2="20.32" width="0.6096" layer="16"/>
-<wire x1="20.32" y1="27.94" x2="13.97" y2="27.94" width="0.6096" layer="1"/>
-<wire x1="10.16" y1="31.75" x2="13.97" y2="27.94" width="0.6096" layer="1"/>
-<wire x1="21.59" y1="26.67" x2="21.59" y2="25.4" width="0.6096" layer="1"/>
-<wire x1="21.59" y1="26.67" x2="20.32" y2="27.94" width="0.6096" layer="1"/>
+<wire x1="10.16" y1="31.75" x2="15.24" y2="31.75" width="0.6096" layer="1"/>
+<wire x1="21.59" y1="25.4" x2="15.24" y2="31.75" width="0.6096" layer="1"/>
 </signal>
 <signal name="N$9">
@@
 <contactref element="SPK." pad="1"/>
 <wire x1="25.4" y1="11.43" x2="24.47115625" y2="11.43" width="0.2032" layer="16"/>
-<wire x1="21.59" y1="5.08" x2="24.13" y2="7.62" width="0.2032" layer="1"/>
-<via x="24.13" y="7.62" extent="1-16" drill="0.35"/>
-<wire x1="24.13" y1="7.62" x2="23.2156" y2="8.5344" width="0.2032" layer="16"/>
-<wire x1="23.2156" y1="8.5344" x2="23.2156" y2="10.16" width="0.2032" layer="16"/>
+<wire x1="21.59" y1="5.08" x2="24.13" y2="5.08" width="0.2032" layer="1"/>
+<via x="24.13" y="5.08" extent="1-16" drill="0.35"/>
+<wire x1="24.13" y1="5.08" x2="23.2156" y2="5.9944" width="0.2032" layer="16"/>
+<wire x1="23.2156" y1="5.9944" x2="23.2156" y2="10.16" width="0.2032" layer="16"/>
 <wire x1="23.2156" y1="10.16" x2="24.4856" y2="11.43" width="0.2032" layer="16"/>
 <wire x1="24.4856" y1="11.43" x2="25.4" y2="11.43" width="0.2032" layer="16"/>
